File: Pcb Files/chase.kicad_sch (KiCad schematic)
At the start: 50 parts, among them P1 Conn_01x01_Pin, P2 Conn_01x01_Pin, P3 Conn_01x01_Pin, P4 Conn_01x01_Pin, P5 Conn_01x01_Pin, P6 Conn_01x01_Pin, P7 Conn_01x01_Pin, P8 Conn_01x01_Pin, P9 Conn_01x01_Pin, Q1 Q_NMOS, Q2 Q_NMOS, Q3 Q_NMOS, U1 ARDUINO_NANO

Commit message: Add files via upload
Parts:
- removed D1, D10, D11, D12, D13, D14, D15, D16, D17, D18, D19, D2, D20, D21, D22, D23, D24, D25, D26, D27, D3, D4, D5, D6, D7, D8, D9: LED, LED_THT:LED_D5.0mm-3, symbol Device:LED
Connections:
- net MOS1: now also U1.10 (D7); no longer U1.24 (A5)
- net MOS2: now also U1.11 (D8); no longer U1.25 (A6)
- net MOS3: now also U1.12 (D9); no longer U1.26 (A7)
- net at L1.1 (Pin_1), Q1.D: no longer U1.10 (D7)
- net at L2.1 (Pin_1), Q2.D: no longer U1.11 (D8)
- net at L3.1 (Pin_1), Q3.D: no longer U1.12 (D9)
Other:
- moved on the sheet: L1, L2, L3
